Commit message: Fixed issues with the vacuum gripper

File: urdf/lite6_fake/lite6_fake_wrapper.urdf.xacro (robot description, xacro)
@@ -82,9 +82,17 @@
       <origin xyz="0 0 0" rpy="0 0 0"/>
     </joint>
+    <!-- Vacuum Gripper Tip Link für das Joint -->
+    <link name="vacuum_tip_link">
+      <inertial>
+        <mass value="0.01"/>
+        <origin xyz="0 0 0" rpy="0 0 0"/>
+        <inertia ixx="0.00001" ixy="0" ixz="0" iyy="0.00001" iyz="0" izz="0.00001"/>
+      </inertial>
+    </link>
     <!-- Virtueller Vacuum Aktor für ros2_control -->
     <joint name="vacuum_joint" type="prismatic">
       <parent link="vacuum_gripper_link"/>
-      <child  link="vacuum_gripper_link"/>
-      <origin xyz="0 0 0" rpy="0 0 0"/>
+      <child  link="vacuum_tip_link"/>
+      <origin xyz="0 0 0.02" rpy="0 0 0"/>
       <axis xyz="0 0 1"/>
       <limit lower="0" upper="1" effort="10" velocity="1"/>
