Commit message: RL Connection available

File: urdf/gripper/authentic_lite6_gripper.urdf.xacro (robot description, xacro)
@@ -67,4 +67,6 @@
       <axis xyz="0 1 0" />
       <limit lower="0" upper="0.015" effort="50" velocity="0.1" />
+      <!-- Realistische Dynamik für bessere Simulation -->
+      <dynamics damping="1.0" friction="0.1"/>
     </joint>
     <!-- Right finger link -->
@@ -101,4 +103,6 @@
       <limit lower="0" upper="0.015" effort="50" velocity="0.1" />
       <mimic joint="${prefix}lite6_left_finger_joint" multiplier="1.0" offset="0.0"/>
+      <!-- Realistische Dynamik für bessere Simulation -->
+      <dynamics damping="1.0" friction="0.1"/>
     </joint>
     <!-- TCP (Tool Center Point) link -->
@@ -109,25 +113,6 @@
       <child link="${prefix}link_tcp" />
     </joint>
-    <!-- ros2_control hardware interface -->
-    <ros2_control name="${prefix}authentic_lite6_gripper_controller" type="system">
-      <hardware>
-        <plugin>mock_components/GenericSystem</plugin>
-      </hardware>
-      <!-- Master joint with command interface -->
-      <joint name="${prefix}lite6_left_finger_joint">
-        <command_interface name="position">
-          <param name="min">0</param>
-          <param name="max">0.015</param>
-        </command_interface>
-        <state_interface name="position"/>
-        <state_interface name="velocity"/>
-        <state_interface name="effort"/>
-      </joint>
-      <!-- Mimic joint (read-only) -->
-      <joint name="${prefix}lite6_right_finger_joint">
-        <state_interface name="position"/>
-        <state_interface name="velocity"/>
-      </joint>
-    </ros2_control>
+    <!-- Gripper wird über das Haupt xArm Hardware-Interface gesteuert -->
+    <!-- Keine separaten ros2_control-Definitionen nötig -->
   </xacro:macro>
 </robot>

File: urdf/lite6_real/lite6_real_wrapper.urdf.xacro (robot description, xacro)
@@ -2,7 +2,6 @@
 <robot xmlns:xacro="http://ros.org/wiki/xacro" name="lite6">
   <!-- ===== Args ===== -->
-  <xacro:arg name="robot_ip"      default="192.168.1.100"/>
+  <xacro:arg name="robot_ip"      default="192.168.1.186"/>
   <xacro:arg name="report_type"   default="dev"/>
-  <xacro:arg name="dof"           default="6"/>
   <xacro:arg name="with_gripper"  default="false"/>
   <xacro:arg name="with_vacuum"   default="false"/>
@@ -28,5 +27,5 @@
   <xacro:property name="mesh_suffix" value="stl"/>
   <xacro:property name="prefix" value="$(arg prefix)"/>
-  <!-- ===== Arm mit echter Hardware (xArmHW Plugin) ===== -->
+  <!-- ===== Arm mit echter Hardware (echtes xArm Hardware Interface) ===== -->
   <xacro:lite6_robot
       prefix="${prefix}"
@@ -34,8 +33,8 @@
       velocity_control="false"
       hard_interface="ros2_control"
-      ros2_control_plugin="xarm_control/XArmHW"
+      ros2_control_plugin="uf_robot_hardware/UFRobotSystemHardware"
       robot_ip="$(arg robot_ip)"
       report_type="$(arg report_type)"
-      dof="$(arg dof)"
+      add_gripper="$(arg with_gripper)"
       kinematics_params_filename="$(arg KIN_YAML)"
       inertial_params_filename="$(arg INERTIAL_YAML)"/>
@@ -107,5 +106,5 @@
     <ros2_control name="vacuum_gripper_controller" type="system">
       <hardware>
-        <plugin>xarm_control/XArmVacuumHW</plugin>
+        <plugin>uf_robot_hardware/UFRobotVacuumHardware</plugin>
         <param name="robot_ip">$(arg robot_ip)</param>
         <param name="report_type">$(arg report_type)</param>
